Commit message: another day another nickle

File: Gazebo/URDF/Segway.urdf (robot description, URDF)
Before this commit: robot segway, 3 links, 2 joints
Links:
- removed link base_link
- added link segway/base_link, mass 0.001; collision box size=0.4 0.4 0.4; visual mesh filename=package://pomdp_ros/Gazebo/Meshes/Segway/Body.stl scale=0.01 0.01 0.01
Joints:
- joint w1_joint: parent base_link -> segway/base_link
- joint w2_joint: parent base_link -> segway/base_link
