Commit message: belief of vehicles done

File: Gazebo/URDF/Flipper.urdf (robot description, URDF)
Before this commit: robot flipper, 1 links, 0 joints
Links:
- removed link world
- added link flipper/base_link, mass 0.001; collision box size=0.4 0.4 0.4; visual mesh filename=package://pomdp_ros/Gazebo/Meshes/Flipper/T-90.stl scale=0.002 0.002 0.002

File: Gazebo/URDF/UAV.urdf (robot description, URDF)
Before this commit: robot uav, 5 links, 4 joints
Links:
- removed link base_link
- added link uav/base_link, mass 0.001; collision box size=0.4 0.4 0.4; visual mesh filename=package://pomdp_ros/Gazebo/Meshes/UAV/Body.stl scale=0.01 0.01 0.01
Joints:
- joint m1_joint: parent base_link -> uav/base_link
- joint m2_joint: parent base_link -> uav/base_link
- joint m3_joint: parent base_link -> uav/base_link
- joint m4_joint: parent base_link -> uav/base_link

File: Gazebo/URDF/cast.urdf (robot description, URDF)
Before this commit: robot cast_flying_arena, 1 links, 0 joints
Links:
- link world: geometry visual mesh filename=package://pomdp_ros/Gazebo/Meshes/cast_simple_2.dae scale=0.0254 0.0254 0.0254

Commit message: changed flipper model out, manual barrier filter working

File: Gazebo/URDF/Flipper.urdf (robot description, URDF)
Before this commit: robot flipper, 1 links, 0 joints
Links:
- link flipper/base_link: geometry collision box size=0.4 0.4 0.4; visual mesh filename=package://pomdp_ros/Gazebo/Meshes/Flipper/Dual.stl scale=0.01 0.01 0.01
